File: battery_board_v3/Battery_Board_V3/Battery_Board_V3.kicad_pcb (KiCad board)
At the start: 4 copper layers, 88 x 94.5 mm, 119 parts, among them IC1 PCA9685PW,118, IC2 LT3652IMSE#PBF, IC3 PCT2075DP,118, J1 Face0, J11 CHARGE, J12 Foot0, J13 Foot1, J14 Foot2, J15 Foot3, J16 RBF, J17 BURN, J18 Bypass, J19 Heater, J2 Face1, J20 Breakout, J3 Face2, J4 Face3, J5 Face4, J6 FC_FACE, K1 APAN3105, Q1 IRF7458, Q2 IRF7458, Q3 MBT2222ADW1T1, Q4 MBT2222ADW1T1, Q5 IRLML2803, Q6 NDS8434, Q7 MMBT2222AT, Q8 IRLML2803, Q9 NDS8434, U1 R5460N208AA, U2 TPS54226PWPRPWP14_2P31X2P46-L, U3 INA219AxD, U4 TCA9548APWR, U5 TPS7A4501DCQT, U6 INA219AxD, U7 1049, U8 1049

Commit message: Better_Battery_Board_with_CAN
Nicole and Freshmen worked on this
Parts:
- removed ? (x2): , 
- added C21: 22pF, Capacitor_SMD:C_0402_1005Metric, F.Cu at (330.7, 128.3)
- added C22: 1uF, Capacitor_SMD:C_0805_2012Metric, F.Cu at (378.4, 121.5)
- added C23: 1uF, Capacitor_SMD:C_0603_1608Metric, F.Cu at (354.1, 136.8)
- added C24: 10uF, Capacitor_SMD:C_0805_2012Metric, F.Cu at (378.4, 124.5)
- added C25: 0.1uF, Capacitor_SMD:C_0402_1005Metric, F.Cu at (330.7, 130.2)
- added C26: 0.1uF, Capacitor_SMD:C_0402_1005Metric, F.Cu at (330.7, 132.2)
- added C27: 0.1uF, Capacitor_SMD:C_0805_2012Metric, F.Cu at (378.4, 127.5)
- added C28: 1uF, Capacitor_SMD:C_0603_1608Metric, F.Cu at (358.1, 109.2)
- added C29: 0.1uF, Capacitor_SMD:C_0402_1005Metric, F.Cu at (333.6, 126.3)
- added C30: 1uF, Capacitor_SMD:C_0603_1608Metric, F.Cu at (358.1, 111.7)
- added C31: 0.1uF, Capacitor_SMD:C_0402_1005Metric, F.Cu at (333.6, 128.3)
- added C32: 0.1uF, Capacitor_SMD:C_0402_1005Metric, F.Cu at (333.6, 130.2)
- added C33: 0.1uF, Capacitor_SMD:C_0402_1005Metric, F.Cu at (333.6, 132.2)
- added C34: 10uF, Capacitor_SMD:C_0603_1608Metric, F.Cu at (358.1, 114.2)
- added C35: 22pf, Capacitor_SMD:C_0402_1005Metric, F.Cu at (336.4, 126.3)
- added C36: 22pf, Capacitor_SMD:C_0402_1005Metric, F.Cu at (336.4, 128.3)
- added C37: 47pf, Capacitor_SMD:C_0402_1005Metric, F.Cu at (336.4, 130.2)
- added C38: 47pf, Capacitor_SMD:C_0402_1005Metric, F.Cu at (336.4, 132.2)
- added C39: 1uF, Capacitor_SMD:C_0603_1608Metric, F.Cu at (358.1, 116.7)
- added C40: 10uF, Capacitor_SMD:C_0603_1608Metric, F.Cu at (358.1, 119.3)
- added C41: 0.1uF, Capacitor_SMD:C_0603_1608Metric, F.Cu at (358.1, 121.8)
- added C42: 0.1uF, Capacitor_SMD:C_0603_1608Metric, F.Cu at (358.1, 124.3)
- added D10: Blue, Diode_SMD:D_0603_1608Metric_Pad1.05x0.95mm_HandSolder, F.Cu at (391.6, 131.2)
- added D6: DFLS130L, Diode_SMD:D_PowerDI-123, F.Cu at (398.9, 133.5)
- added D7: D_Schottky, Diode_SMD:D_SMB, F.Cu at (423.0, 46.9)
- added D8: NSR0320, Diode_SMD:D_SOD-323F, F.Cu at (323.4, 135.2)
- added D9: DFLS130L, Diode_SMD:D_PowerDI-123, F.Cu at (398.9, 137.2)
- added FB1: FerriteBead, Resistor_SMD:R_0603_1608Metric, F.Cu at (358.1, 126.8)
- added FB2: FerriteBead, Resistor_SMD:R_0603_1608Metric, F.Cu at (358.1, 129.3)
- added FB3: FerriteBead, Resistor_SMD:R_0603_1608Metric, F.Cu at (358.1, 131.8)
- added IC4: LT3652IMSE#PBF, Package_SO:MSOP-12-1EP_3x4mm_P0.65mm_EP1.65x2.85mm, F.Cu at (413.5, 77.9)
- added J10: Face0, Battery Board:MOLEX_5040500591, F.Cu at (402.1, 26.3)
- added J21: CAN1, Connector_JST:JST_SH_SM04B-SRSS-TB_1x04-1MP_P1.00mm_Horizontal, F.Cu at (530.9, 56.3)
- added J22: BM04B-SRSS-TB(LF)(SN), Battery Board:JST_BM04B-SRSS-TB(LF)(SN), F.Cu at (424.4, 89.5)
- added J23: CAN2, Connector_JST:JST_SH_SM04B-SRSS-TB_1x04-1MP_P1.00mm_Horizontal, F.Cu at (407.1, 108.1)
- added J24: Conn_ARM_JTAG_SWD_10, Battery Board:JTAG_2X05_1.27MM_BOX_NOCREAM, F.Cu at (492.7, 39.9)
- added J25: Life Makes Lemonade, Connector_PinHeader_2.54mm:PinHeader_1x06_P2.54mm_Vertical, F.Cu at (412.2, 23.6)
- added J26: BM04B-SRSS-TB(LF)(SN), Battery Board:JST_BM04B-SRSS-TB(LF)(SN), F.Cu at (424.4, 95.8)
- added J27: USB_B_Micro, FC_DEV_BOARD:MOLEX_105164-0001, F.Cu at (472.6, 4.79)
- added J7: Foot2, Battery Board:MOLEX_504050-0291, F.Cu at (337.8, 121.5)
- added J8: Foot3, Battery Board:MOLEX_504050-0291, F.Cu at (347.4, 112.8)
- added J9: RBF, Battery Board:MOLEX_504050-0291, F.Cu at (347.4, 121.5)
- added JP2: SolderJumper_2_Open, Jumper:SolderJumper-2_P1.3mm_Open_RoundedPad1.0x1.5mm, F.Cu at (391.4, 134.5)
- added LED1: WS2812B_SK6812_1515, LED_SMD:LED_WS2812B_PLCC4_5.0x5.0mm_P3.2mm, F.Cu at (423.3, 131.9)
- added R45: 120, Resistor_SMD:R_0603_1608Metric, F.Cu at (374.2, 116.7)
- added R46: 10K, Resistor_SMD:R_0603_1608Metric, F.Cu at (374.2, 119.3)
- added R47: 10k, Resistor_SMD:R_Array_Convex_4x1206, F.Cu at (416.3, 132.0)
- added R48: 0.002, Resistor_SMD:R_2512_6332Metric, F.Cu at (415.9, 88.8)
- added R49: 0.002, Resistor_SMD:R_2512_6332Metric, F.Cu at (415.9, 93.6)
- added R50: 634k, Resistor_SMD:R_0603_1608Metric, F.Cu at (374.2, 121.8)
- added R51: 412k, Resistor_SMD:R_0603_1608Metric, F.Cu at (374.2, 124.3)
- added R52: 22, Resistor_SMD:R_0603_1608Metric, F.Cu at (473.0, 16.6)
- added R53: 22, Resistor_SMD:R_0603_1608Metric, F.Cu at (474.7, 14.9)
- added R54: 0.1, Resistor_SMD:R_2512_6332Metric, F.Cu at (415.9, 98.5)
- added R55: 1k, Resistor_SMD:R_0603_1608Metric, F.Cu at (374.2, 131.8)
- added R56: 10k, Resistor_SMD:R_0603_1608Metric, F.Cu at (374.2, 134.3)
- added SW1: KMR2, Battery Board:BTN_KMR2_4.6X2.8, F.Cu at (347.8, 127.4)
- added SW2: KMR2, Battery Board:BTN_KMR2_4.6X2.8, F.Cu at (347.8, 131.7)
- added TP7: RESET, TestPoint:TestPoint_Loop_D1.80mm_Drill1.0mm_Beaded, F.Cu at (419.0, 121.7)
- added TP8: TestPoint, TestPoint:TestPoint_Loop_D1.80mm_Drill1.0mm_Beaded, F.Cu at (418.9, 126.3)
- added U10: MCP25625-E/ML, Package_DFN_QFN:QFN-28-1EP_6x6mm_P0.65mm_EP4.25x4.25mm, F.Cu at (530.8, 47.0)
- added U11: INA219AxD, Package_SO:SOIC-8_3.9x4.9mm_P1.27mm, F.Cu at (398.5, 110.4)
- added U12: MAX706RESA, Package_SO:SO-8_3.9x4.9mm_P1.27mm, F.Cu at (398.5, 116.9)
- added U13: INA219AxD, Package_SO:SOIC-8_3.9x4.9mm_P1.27mm, F.Cu at (398.5, 123.3)
- added U9: TLVH431 DBZ SOT-23, Package_TO_SOT_SMD:SOT-23, F.Cu at (422.3, 78.0)
- added Y1: 12MHZ, Crystal:Crystal_SMD_2520-4Pin_2.5x2.0mm, F.Cu at (425.6, 32.3)
- added Y2: 16MHZ 12 pf, Crystal:Crystal_SMD_2520-4Pin_2.5x2.0mm, F.Cu at (425.6, 36.4)
- C13: value 200uF -> 10uF; footprint Capacitor_SMD:C_1210_3225Metric -> Capacitor_SMD:C_0603_1608Metric
- C14: value 0.1uF -> 200uF; footprint Capacitor_SMD:C_0603_1608Metric -> Capacitor_SMD:C_1210_3225Metric
- C15: value 10uF -> 200uF; footprint Capacitor_SMD:C_0603_1608Metric -> Capacitor_SMD:C_1210_3225Metric
- C16: footprint Capacitor_SMD:C_0603_1608Metric -> Capacitor_SMD:C_0805_2012Metric
- C17: value 1uF -> 0.01uF; footprint Capacitor_SMD:C_0603_1608Metric -> Capacitor_SMD:C_0805_2012Metric
- C18: value 10uF -> 0.1uF; footprint Capacitor_SMD:C_0603_1608Metric -> Capacitor_SMD:C_0805_2012Metric
- C19: value 200uF -> 0.01uF; footprint Capacitor_SMD:C_1210_3225Metric -> Capacitor_SMD:C_0805_2012Metric
- C20: value 0.1uF -> 22pF; footprint Capacitor_SMD:C_0603_1608Metric -> Capacitor_SMD:C_0402_1005Metric
- D1: value D_Schottky -> DFLS130L; footprint CMSH3-40MA:DIOM5226X262N -> Diode_SMD:D_PowerDI-123
- D2: value DFLS130L -> green; footprint MaxLib:PWRDI-123 -> Diode_SMD:D_0603_1608Metric_Pad1.05x0.95mm_HandSolder
- D3: value D_Schottky -> red; footprint CMSH3-40MA:DIOM5226X262N -> Diode_SMD:D_0603_1608Metric_Pad1.05x0.95mm_HandSolder
- D4: value DFLS130L -> D_Schottky; footprint MaxLib:PWRDI-123 -> Diode_SMD:D_SMB
- D5: value DFLS130L -> PESD1CAN; footprint MaxLib:PWRDI-123 -> Package_TO_SOT_SMD:SOT-23-3
- IC2: value LT3652IMSE#PBF -> PCT2075DP,118; footprint LT3652IMSE:SOP65P490X110-13N -> Package_SO:TSSOP-8_3x3mm_P0.65mm
- IC3: value PCT2075DP,118 -> RP2040_QFN56; footprint Package_SO:TSSOP-8_3x3mm_P0.65mm -> Package_DFN_QFN:QFN-56-1EP_7x7mm_P0.4mm_EP3.2x3.2mm
- J1: value Face0 -> Bypass; footprint MOLEX PICO LOCK 5 POS:MOLEX_5040500591 -> Connector_PinSocket_2.54mm:PinSocket_1x02_P2.54mm_Vertical
- J11: value CHARGE -> Face1; footprint MOLEX PICO LOCK 2 POS:MOLEX_504050-0291 -> Battery Board:MOLEX_5040500591
- J12: value Foot0 -> Face2; footprint MOLEX PICO LOCK 2 POS:MOLEX_504050-0291 -> Battery Board:MOLEX_5040500591
- J13: value Foot1 -> Face3; footprint MOLEX PICO LOCK 2 POS:MOLEX_504050-0291 -> Battery Board:MOLEX_5040500591
- J14: value Foot2 -> Face4; footprint MOLEX PICO LOCK 2 POS:MOLEX_504050-0291 -> Battery Board:MOLEX_5040500591
- J15: value Foot3 -> Face4; footprint MOLEX PICO LOCK 2 POS:MOLEX_504050-0291 -> Battery Board:MOLEX_5040500591
- J16: value RBF -> Breakout; footprint MOLEX PICO LOCK 2 POS:MOLEX_504050-0291 -> Connector_JST:JST_SH_SM04B-SRSS-TB_1x04-1MP_P1.00mm_Horizontal
- J17: value BURN -> Screw_Terminal_01x02; footprint MOLEX PICO LOCK 2 POS:MOLEX_504050-0291 -> TerminalBlock:TerminalBlock_bornier-2_P5.08mm
- J18: value Bypass -> I2C; footprint Connector_PinSocket_2.54mm:PinSocket_1x02_P2.54mm_Vertical -> Connector_JST:JST_SH_SM04B-SRSS-TB_1x04-1MP_P1.00mm_Horizontal
- J19: value Heater -> Screw_Terminal_01x02; footprint MOLEX PICO LOCK 2 POS:MOLEX_504050-0291 -> Battery Board:ScrewTerminal
- J2: value Face1 -> Heater; footprint MOLEX PICO LOCK 5 POS:MOLEX_5040500591 -> Battery Board:MOLEX_504050-0291
- J20: value Breakout -> BM04B-SRSS-TB(LF)(SN); footprint SM04B-SRSS-TB_LF__SN_:JST_SM04B-SRSS-TB(LF)(SN) -> Battery Board:JST_BM04B-SRSS-TB(LF)(SN)
- J3: value Face2 -> BURN; footprint MOLEX PICO LOCK 5 POS:MOLEX_5040500591 -> Battery Board:MOLEX_504050-0291
- J4: value Face3 -> CHARGE; footprint MOLEX PICO LOCK 5 POS:MOLEX_5040500591 -> Battery Board:MOLEX_504050-0291
- J5: value Face4 -> Foot0; footprint MOLEX PICO LOCK 5 POS:MOLEX_5040500591 -> Battery Board:MOLEX_504050-0291
- J6: value FC_FACE -> Foot1; footprint Connector_Molex:Molex_Pico-Lock_504050-1291_1x12-1MP_P1.50mm_Horizontal -> Battery Board:MOLEX_504050-0291
- JP1: value Jumper_3_Bridged12 -> SolderJumper_3_Open; footprint MaxLib:SolderJumper-3_P1.3mm_Bridged12_RoundedPad1.0x1.5mm -> Jumper:SolderJumper-3_P1.3mm_Open_RoundedPad1.0x1.5mm_NumberLabels
- Q4: value MBT2222ADW1T1 -> MMBT2222AT; footprint Package_TO_SOT_SMD:SOT-363_SC-70-6 -> Package_TO_SOT_SMD:SOT-523
- Q5: value IRLML2803 -> MBT2222ADW1T1; footprint MaxLib:SOT-23 -> Package_TO_SOT_SMD:SOT-363_SC-70-6
- Q6: value NDS8434 -> IRLML2803; footprint MaxLib:NDS8434 -> Package_TO_SOT_SMD:SOT-23
- Q7: value MMBT2222AT -> IRLML2803; footprint Package_TO_SOT_SMD:SOT-523 -> Package_TO_SOT_SMD:SOT-23
- Q8: value IRLML2803 -> NDS8434; footprint MaxLib:SOT-23 -> Package_SO:SOIC-8-1EP_3.9x4.9mm_P1.27mm_EP2.514x3.2mm
- Q9: footprint MaxLib:NDS8434 -> Package_SO:SOIC-8-1EP_3.9x4.9mm_P1.27mm_EP2.514x3.2mm
- R10: value 20K -> 100K
- R12: value 100K -> 20K
- R14: value 10k -> 100K
- R15: value 10K -> 100K
- R16: value 4.7k -> 10k; footprint Resistor_SMD:R_0603_1608Metric -> Resistor_SMD:R_Array_Convex_4x1206
- R17: value 100k -> 10K
- R18: value 10K -> 10k; footprint Resistor_SMD:R_0603_1608Metric -> Resistor_SMD:R_Array_Convex_4x1206
- R19: value 10K -> 634k
- R2: value 1K -> 10K
- R21: value 10K -> 10k
- R22: value 0.002 -> 10k; footprint Resistor_SMD:R_2512_6332Metric -> Resistor_SMD:R_0603_1608Metric
- R23, R24: value 10K -> 4.7k
- R26: value 10K -> 3.3K
- R27, R28: value 10K -> 100k
- R3: value 330 -> 1K
- R31: value 3.3K -> 1-MOhm
- R32: value 200k -> 100-Ohm
- R33: value 85k -> 100-Ohm
- R34: value 634k -> 10k-Ohm
- R35: value 412k -> 10k
- R36: value 0.1 -> 1k; footprint Resistor_SMD:R_2512_6332Metric -> Resistor_SMD:R_0603_1608Metric
- R37: value 0.002 -> 1k; footprint Resistor_SMD:R_2512_6332Metric -> Resistor_SMD:R_0603_1608Metric
- R38: value 10K -> 1k
- R40: value 10k -> 1k
- R41: value 4.7k -> 10k
- R42: value 100k -> 200k
- R43: value 10K -> 85k
- R44: value 634k -> 10k
- R5: value 73.2K -> 330
- R7: value 22.1K -> 73.2K
- R8: value 100K -> 22.1K
- R9: value 100K -> 10k
- U1: footprint R5460N233AF:R5460N233AF-SOT95P280X130-6N -> Package_TO_SOT_SMD:SOT-23-6
- U2: value TPS54226PWPRPWP14_2P31X2P46-L -> 1049; footprint MaxLib:PWP14_2P31X2P46-L -> 1049:1049; moved to B.Cu
- U3: value INA219AxD -> TPS54226PWPRPWP14_2P31X2P46-L; footprint Package_SO:SOIC-8_3.9x4.9mm_P1.27mm -> Package_SO:HTSSOP-14-1EP_4.4x5mm_P0.65mm_EP3.4x5mm_Mask3x3.1mm_ThermalVias
- U4: value TCA9548APWR -> 1049; footprint TCA9548APWR:SOP65P640X120-24N -> 1049:1049; moved to B.Cu
- U5: value TPS7A4501DCQT -> TCA9548APWR; footprint MaxLib:TPS7A4501DCQT -> TCA9548APWR:SOP65P640X120-24N
- U6: value INA219AxD -> TPS7A4501DCQT; footprint Package_SO:SOIC-8_3.9x4.9mm_P1.27mm -> Package_TO_SOT_SMD:SOT-223-6
- U7: value 1049 -> ADS1015IDGS; footprint 1049:1049 -> Package_SO:TSSOP-10_3x3mm_P0.5mm; moved to F.Cu
- U8: value 1049 -> AD8495; footprint 1049:1049 -> Package_SO:MSOP-8_3x3mm_P0.65mm; moved to F.Cu
- moved IC3 332.8 mm to (481.5, 24.9), turned to 45 degrees
- moved J17 304.1 mm to (417.8, 25.8), turned to 0 degrees
- moved IC1 298.9 mm to (414.3, 44.3), turned to 0 degrees
- moved TP6 297.9 mm to (414.3, 126.3)
- moved J20 295.7 mm to (424.4, 83.1)
- moved D5 295.2 mm to (423.9, 121.6)
- moved Q6 291.3 mm to (422.3, 69.1), turned to 0 degrees
- moved Q7 282.3 mm to (422.3, 73.5), turned to 0 degrees
- moved U3 273.9 mm to (418.9, 33.7)
- moved J19 273.8 mm to (384.9, 129.4), turned to 0 degrees
- moved U5 273.7 mm to (415.0, 54.6)
- moved J12 271.7 mm to (402.1, 46.3), turned to 0 degrees
- moved R16 271.5 mm to (405.4, 132.0)
- moved TP3 270.8 mm to (409.7, 121.7)
- moved K1 268.9 mm to (405.1, 114.8), turned to 0 degrees
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Connections:
- C10 pad 1: Net-(C10-Pad1) -> Net-(U3-SS)
- C11 pad 1: Net-(C11-Pad1) -> Net-(U3-VREG5)
- C12 pad 1: Net-(C12-Pad1) -> Net-(Q5A-C1)
- C12 pad 2: Net-(C12-Pad2) -> Net-(Q3B-B2)
- C13 pad 1: BURN -> GND
- C13 pad 2: GND -> /V_RF
- C14 pad 1: GND -> BURN
- C14 pad 2: +3V3 -> GND
- C15 pad 1: GND -> Heater
- C15 pad 2: /V_RF -> GND
- C16 pad 1: Net-(C16-Pad1) -> AVDD
- C16 pad 2: GND -> AGND
- C17 pad 1: Net-(C17-Pad1) -> GND
- C17 pad 2: Net-(C17-Pad2) -> Net-(U8--IN)
- C18 pad 1: PACK+ -> Net-(U8-+IN)
- C18 pad 2: GND -> Net-(U8--IN)
- C19 pad 1: Heater -> Net-(U8-+IN)
- C20 pad 2: +3V3 -> Net-(IC3-XIN)
- C6 pad 1: Net-(C6-Pad1) -> Net-(U3-SW1)
- C6 pad 2: Net-(C6-Pad2) -> Net-(U3-VBST)
- C7 pad 2: Net-(C7-Pad2) -> Net-(U1-V-)
- C8 pad 2: Net-(C8-Pad2) -> Net-(U1-VC)
- D2 pad A: PACK+ -> FC_TX
- D2 pad C: Net-(C17-Pad2) -> Net-(D2-PadC)
- IC1 pad 12: unconnected-(IC1-Pad12) -> FC_RESET
- IC1 pad 26: SCL_MAIN -> SCL0
- IC1 pad 27: SDA_MAIN -> SDA0
- IC2 pad 1: Net-(C16-Pad1) -> SDA0
- IC2 pad 2: Net-(IC2-Pad2) -> SCL0
- IC2 pad 3: Net-(C16-Pad1) -> Net-(IC2-OS)
- IC2 pad 4: CHRG' -> GND
- IC2 pad 5: unconnected-(IC2-Pad5) -> +3V3
- IC2 pad 6: GND -> +3V3
- IC2 pad 7: Net-(IC2-Pad7) -> +3V3
- IC2 pad 8: unconnected-(IC2-Pad8) -> +3V3
- IC3 pad 1: SDA_MAIN -> +3V3
- IC3 pad 2: SCL_MAIN -> FC_RX
- IC3 pad 3: Net-(IC3-Pad3) -> FC_TX
- IC3 pad 4: GND -> SDA1
- IC3 pad 5: +3V3 -> SCL1
- IC3 pad 6: +3V3 -> SDA0
- IC3 pad 7: +3V3 -> SCL0
- IC3 pad 8: +3V3 -> ENABLE_BURN
- J1 pad 1: VSOLAR -> VBATT_SENSE
- J1 pad 2: GND -> VBatt
- J11 pad 1: GND -> VSOLAR
- J11 pad 2: PACK+ -> GND
- J12 pad 1: Net-(J12-Pad1) -> VSOLAR
- J12 pad 2: VBatt -> GND
- J13 pad 1: VBatt1 -> VSOLAR
- J13 pad 2: Net-(J12-Pad1) -> GND
- J14 pad 1: Net-(J14-Pad1) -> VSOLAR
- J14 pad 2: VBatt -> GND
- J15 pad 1: VBatt1 -> +5V
- J15 pad 2: Net-(J14-Pad1) -> GND
- J16 pad 1: VBATT_SENSE -> GND
- J16 pad 2: VBatt1 -> +3V3
- J17 pad 1: GND -> Net-(J17-Pin_1)
- J17 pad 2: BURN -> Net-(J17-Pin_2)
- J18 pad 1: VBATT_SENSE -> GND
- J18 pad 2: VBatt -> +3V3
- J19 pad 1: GND -> Net-(J17-Pin_2)
- J19 pad 2: Heater -> Net-(J17-Pin_1)
- J2 pad 1: VSOLAR -> GND
- J2 pad 2: GND -> Heater
- J20 pad 1: GND -> +3V3
- J20 pad 2: +3V3 -> GND
- J20 pad 3: Break_SDA -> +5V
- J20 pad 4: Break_SCL -> GND
- J20 pad S1: (no net) -> GND
- J20 pad S2: (no net) -> GND
- J3 pad 1: VSOLAR -> GND
- J3 pad 2: GND -> BURN
- J4 pad 1: VSOLAR -> GND
- J4 pad 2: GND -> PACK+
- J5 pad 1: VSOLAR -> Net-(J5-Pin_1)
- J5 pad 2: GND -> VBatt
- J6 pad 1: GND -> VBatt1
- J6 pad 2: VCC_RF1 -> Net-(J5-Pin_1)
- JP1 pad 1: /V_RF -> +3V3
- JP1 pad 2: VCC_RF1 -> +5V
- JP1 pad 3: +3V3 -> /V_RF
- K1 pad C2: Net-(D5-PadA) -> Net-(Q4-C)
- L1 pad 1: Net-(C6-Pad1) -> Net-(U3-SW1)
- L2 pad 1: Net-(C17-Pad1) -> Net-(D7-K)
- L2 pad 2: Net-(IC2-Pad10) -> Net-(IC4-SENSE)
- Q3 pad 2: Net-(Q3-Pad2) -> Net-(Q3A-B1)
- Q3 pad 3: Net-(Q3-Pad2) -> Net-(Q3A-B1)
- Q3 pad 5: Net-(C12-Pad2) -> Net-(Q3B-B2)
- Q4 pad 1: GND -> BURN_RELAY_A
- Q4 pad 2: Net-(Q4-Pad2) -> GND
- Q4 pad 3: Net-(C12-Pad1) -> Net-(Q4-C)
- Q5 pad 1: Net-(Q5-Pad1) -> GND
- Q5 pad 2: GND -> Net-(Q5A-B1)
- Q5 pad 3: Net-(Q5-Pad3) -> Net-(Q5A-C1)
- Q6 pad 1: Net-(K1-PadNO) -> Net-(Q6-G)
- Q6 pad 2: Net-(K1-PadNO) -> GND
- Q6 pad 3: Net-(K1-PadNO) -> Net-(Q6-D)
- Q7 pad 1: BURN_RELAY_A -> Net-(Q7-G)
- Q7 pad 3: Net-(D5-PadA) -> Net-(Q7-D)
- Q8 pad 1: Net-(Q8-Pad1) -> Net-(K1-PadNO)
- Q8 pad 2: GND -> Net-(K1-PadNO)
- Q8 pad 3: Net-(Q8-Pad3) -> Net-(K1-PadNO)
- Q9 pad 4: Net-(Q8-Pad3) -> Net-(Q7-D)
- R10 pad 1: Net-(Q4-Pad2) -> VBUSP
- R10 pad 2: Net-(Q3-Pad2) -> Net-(Q3A-B1)
- R11 pad 1: VBUSP -> Net-(U3-PG)
- R11 pad 2: Net-(R11-Pad2) -> Net-(U3-VREG5)
- R12 pad 1: Net-(R11-Pad2) -> Net-(Q5A-B1)
- R12 pad 2: Net-(C12-Pad2) -> Net-(Q3A-B1)
- R13 pad 2: Net-(C12-Pad1) -> Net-(R13-Pad2)
- R14 pad 1: ENAB_BURN -> Net-(R13-Pad2)
- R14 pad 2: GND -> Net-(Q3B-B2)
- R15 pad 1: Net-(Q4-Pad5) -> VBUSP
- R15 pad 2: VBUS_RESET -> Net-(Q5A-C1)
- R16 pad 1: Net-(Q5-Pad1) -> F3_SDA
- R16 pad 2: ENAB_BURN -> F2_SDA
- R17 pad 1: Net-(Q5-Pad3) -> Net-(Q5B-B2)
- R17 pad 2: Net-(K1-PadNO) -> VBUS_RESET
- R18 pad 1: +3V3 -> F3_SCL
- R18 pad 2: F3_SDA -> F2_SCL
- R19 pad 1: +3V3 -> GND
- R19 pad 2: F2_SDA -> Net-(K1-PadNO)
- R2 pad 1: Net-(C7-Pad2) -> +3V3
- R2 pad 2: GND -> Net-(IC2-OS)
- R20 pad 2: F1_SDA -> I2C_RESET
- R21 pad 1: +3V3 -> ENAB_BURN
- R21 pad 2: F0_SDA -> GND
- R22 pad 1: VBUSP -> ENAB_HEATER
- R22 pad 2: VBATT_SENSE -> GND
- R23 pad 1: +3V3 -> Net-(Q6-G)
- R23 pad 2: F3_SCL -> ENAB_BURN
- R24 pad 1: +3V3 -> Net-(Q7-G)
- R24 pad 2: I2C_RESET -> ENAB_HEATER
- R25 pad 1: +3V3 -> /V_RF
- R25 pad 2: F2_SCL -> Net-(U6-SENSE/ADJ)
- R26 pad 1: +3V3 -> Net-(U6-SENSE/ADJ)
- R26 pad 2: F1_SCL -> GND
- R27 pad 1: +3V3 -> Net-(Q6-D)
- R27 pad 2: F0_SCL -> Net-(K1-PadNO)
- R28 pad 1: +3V3 -> Net-(Q7-D)
- R28 pad 2: F4_SCL -> Net-(K1-PadNO)
- R29 pad 2: F4_SDA -> F4_SCL
- R3 pad 1: BM -> Net-(U1-V-)
- R3 pad 2: Net-(C8-Pad2) -> GND
- R30 pad 1: /V_RF -> +3V3
- R30 pad 2: Net-(R30-Pad2) -> F4_SDA
- R31 pad 1: Net-(R30-Pad2) -> Net-(J17-Pin_1)
- R32 pad 1: Net-(C16-Pad1) -> Net-(J17-Pin_2)
- R32 pad 2: Net-(IC2-Pad2) -> Net-(U8--IN)
- R33 pad 1: GND -> Net-(U8-+IN)
- R33 pad 2: Net-(IC2-Pad2) -> Net-(J17-Pin_1)
- R34 pad 1: Net-(IC2-Pad7) -> GND
- R34 pad 2: PACK+ -> Net-(JP2-A)
- R35 pad 1: GND -> +3V3
- R35 pad 2: Net-(IC2-Pad7) -> /~{RESET}
- R36 pad 1: PACK+ -> Net-(U8-REF)
- R36 pad 2: Net-(IC2-Pad10) -> Net-(U8-+Vs)
- R37 pad 1: VSOLAR_I -> Net-(IC3-XOUT)
- R37 pad 2: VSOLAR -> Net-(C21-Pad2)
- R38 pad 1: +3V3 -> Net-(D2-PadC)
- R38 pad 2: Net-(IC3-Pad3) -> GND
- R39 pad 1: BURN_RELAY_A -> +3V3
- R39 pad 2: GND -> Net-(U10-RESET)
- R4 pad 1: PACK+ -> BM
- R4 pad 2: /VDD -> Net-(U1-VC)
- R40 pad 1: ENAB_HEATER -> Net-(D3-PadC)
- R41 pad 1: Net-(Q8-Pad1) -> +3V3
- R41 pad 2: ENAB_HEATER -> SPI0_CS0
- R42 pad 1: Net-(Q8-Pad3) -> Net-(D4-K)
- R42 pad 2: Net-(K1-PadNO) -> Net-(IC4-VIN_REG)
- R43 pad 1: +3V3 -> GND
- R43 pad 2: CHRG' -> Net-(IC4-VIN_REG)
- R44 pad 1: GND -> /~{RESET}
- R44 pad 2: Net-(K1-PadNO) -> Net-(U12-~{RESET})
- R5 pad 1: Net-(R5-Pad1) -> PACK+
- R5 pad 2: +3V3 -> /VDD
- R6 pad 1: VBUSP -> Net-(U3-VFB)
- R6 pad 2: /3V3_EN -> +3V3
- R7 pad 1: GND -> VBUSP
- R7 pad 2: Net-(R5-Pad1) -> /3V3_EN
- R8 pad 1: VBUSP -> GND
- R8 pad 2: Net-(Q3-Pad2) -> Net-(U3-VFB)
- R9 pad 1: Net-(R9-Pad1) -> BURN_RELAY_A
- R9 pad 2: Net-(C11-Pad1) -> GND
- TP1 pad 1: B- -> +3V3
- TP2 pad 1: BM -> B-
- TP3 pad 1: GND -> BM
- TP4 pad 1: PACK+ -> GND
- TP5 pad 1: +3V3 -> PACK+
- U1 pad 3: Net-(C7-Pad2) -> Net-(U1-V-)
- U1 pad 4: Net-(C8-Pad2) -> Net-(U1-VC)
- U2 pad 1: +3V3 -> unconnected-(U2-Pad1)
- U2 pad 2: Net-(R5-Pad1) -> unconnected-(U2-Pad2)
- U2 pad 3: Net-(C11-Pad1) -> unconnected-(U2-Pad3)
- U2 pad 4: Net-(C10-Pad1) -> unconnected-(U2-Pad4)
- U2 pad 5: GND -> unconnected-(U2-Pad5)
- U2 pad 6: Net-(R9-Pad1) -> B-
- U2 pad 7: /3V3_EN -> B-
- U2 pad 8: GND -> BM
- U2 pad 9: GND -> BM
- U3 pad 1: GND -> +3V3
- U3 pad 2: GND -> Net-(U3-VFB)
- U3 pad 3: SDA_MAIN -> Net-(U3-VREG5)
- U3 pad 4: SCL_MAIN -> Net-(U3-SS)
- U3 pad 5: +3V3 -> GND
- U3 pad 6: GND -> Net-(U3-PG)
- U3 pad 7: VBUSP -> /3V3_EN
- U3 pad 8: VBATT_SENSE -> GND
- U4 pad 1: +3V3 -> unconnected-(U4-Pad1)
- U4 pad 2: +3V3 -> unconnected-(U4-Pad2)
- U4 pad 3: I2C_RESET -> unconnected-(U4-Pad3)
- U4 pad 4: F0_SDA -> unconnected-(U4-Pad4)
- U4 pad 5: F0_SCL -> unconnected-(U4-Pad5)
- U4 pad 6: F1_SDA -> BM
- U4 pad 7: F1_SCL -> BM
- U4 pad 8: F2_SDA -> PACK+
- U4 pad 9: F2_SCL -> PACK+
- U5 pad 1: ENAB_RF -> +3V3
- U5 pad 2: VBUSP -> +3V3
- U5 pad 3: GND -> I2C_RESET
- U5 pad 4: /V_RF -> F0_SDA
- U5 pad 5: Net-(R30-Pad2) -> F0_SCL
- U5 pad 6: GND -> F1_SDA
- U6 pad 1: +3V3 -> ENAB_RF
- U6 pad 2: GND -> VBUSP
- U6 pad 3: SDA_MAIN -> GND
- U6 pad 4: SCL_MAIN -> /V_RF
- U6 pad 5: +3V3 -> Net-(U6-SENSE/ADJ)
- U7 pad 1: unconnected-(U7-Pad1) -> Net-(JP2-A)
- U7 pad 3: unconnected-(U7-Pad3) -> AGND
- U7 pad 4: unconnected-(U7-Pad4) -> AVDD
- U7 pad 5: unconnected-(U7-Pad5) -> OUT
- U7 pad 6: B- -> AVDD
- U7 pad 7: B- -> AVDD
- U7 pad 8: BM -> AVDD
- U7 pad 9: BM -> SDA0
- U8 pad 1: unconnected-(U8-Pad1) -> Net-(U8--IN)
- U8 pad 2: unconnected-(U8-Pad2) -> Net-(U8-REF)
- U8 pad 3: unconnected-(U8-Pad3) -> GND
- U8 pad 5: unconnected-(U8-Pad5) -> OUT
- U8 pad 6: BM -> OUT
- U8 pad 7: BM -> Net-(U8-+Vs)
- U8 pad 8: PACK+ -> Net-(U8-+IN)
Routing:
- net GND: track 270.5 -> 0.00 mm, vias 55 -> 0
- net VBUSP: track 172.0 -> 0.00 mm, vias 18 -> 0
- net PACK+: track 173.8 -> 19.1 mm, vias 2 -> 0
- net +3V3: track 142.8 -> 0.00 mm, vias 22 -> 0
- net VSOLAR: track 140.8 -> 0.00 mm, vias 4 -> 0
- net F0_ENB: track 122.8 -> 0.00 mm, vias 4 -> 0
- net F1_ENB: track 104.1 -> 0.00 mm, vias 2 -> 0
- net SDA_MAIN: track 92.5 -> 0.00 mm, vias 8 -> 0
- net F2_ENB: track 90.6 -> 0.00 mm
- net SCL_MAIN: track 89.4 -> 0.00 mm, vias 8 -> 0
- net BURN_RELAY_A: track 83.2 -> 0.00 mm, vias 4 -> 0
- net B-: track 99.5 -> 19.1 mm, vias 1 -> 0
- net F3_SDA: track 74.9 -> 0.00 mm, vias 6 -> 0
- net F3_SCL: track 73.6 -> 0.00 mm, vias 6 -> 0
- net ENAB_BURN: track 71.6 -> 0.00 mm, vias 4 -> 0
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- removed copper zone on F.Cu, net +3V3
- removed copper zone on F.Cu, net VBUSP
