File: battery_board_v3/Battery_Board_V3/Battery_Board_V3.kicad_sch (KiCad schematic)
At the start: 145 parts, among them IC1 PCA9685PW,118, IC2 LT3652IMSE#PBF, IC3 PCT2075DP,118, J1 Face0, J11 CHARGE, J12 Foot0, J13 Foot1, J14 Foot2, J15 Foot3, J16 RBF, J17 BURN, J18 Bypass, J19 Heater, J2 Face1, J3 Face2, J4 Face3, J5 Face4, J6 FC_FACE, J7 Breakout, K1 APAN3105, Q1 IRF7458, Q2 IRF7458, Q3 MBT2222ADW1T1, Q4 MBT2222ADW1T1, Q5 IRLML2803, Q6 NDS8434, Q7 MMBT2222AT, Q8 IRLML2803, Q9 NDS8434, U1 R5460N208AA, U2 TPS54226PWPRPWP14_2P31X2P46-L, U3 INA219AxD, U4 TCA9548APWR, U5 TPS7A4501DCQT, U6 INA219AxD, U7 1049, U8 1049

Commit message: Better_Battery_Board_with_CAN
Nicole and Freshmen worked on this
Parts:
- removed J6: FC_FACE, Connector_Molex:Molex_Pico-Lock_504050-1291_1x12-1MP_P1.50mm_Horizontal, symbol Connector_Generic:Conn_01x12
- removed J?: BATT_ADD_IN, symbol Connector_Generic:Conn_01x04
- removed J?: BAT_ADD_OUT, symbol Connector_Generic:Conn_01x04
- removed JP1: Jumper_3_Bridged12, MaxLib:SolderJumper-3_P1.3mm_Bridged12_RoundedPad1.0x1.5mm, symbol mainboard-rescue:Jumper_3_Bridged12-Jumper
- removed TP?: TESTPOINTROUND1.5MMNO, Adafruit ItsyBitsy RP2040:TESTPOINT_ROUND_1.5MM_NO, symbol Adafruit ItsyBitsy RP2040-eagle-import:TESTPOINTROUND1.5MMNO
- removed U?: CAT24C208WI-GT3, SOIC8_ONS, symbol CAT24C208WI-GT3:CAT24C208WI-GT3
- removed X?: microUSB, Molex USB Micro B:MOLEX_105164-0001, symbol Adafruit ItsyBitsy RP2040-eagle-import:USB_MICRO_NARROW
- added C13 (x2): 47pf, Capacitor_SMD:C_0402_1005Metric, symbol Adafruit Ethernet FeatherWing-eagle-import:CAP_CERAMIC0603_NO
- added C13 (x2): 22pf, Capacitor_SMD:C_0402_1005Metric, symbol Adafruit Ethernet FeatherWing-eagle-import:CAP_CERAMIC0603_NO
- added C16, C24: 10uF, Capacitor_SMD:C_0805_2012Metric, symbol Device:C
- added C17, C19: 0.01uF, Capacitor_SMD:C_0805_2012Metric, symbol Device:C
- added C18, C27: 0.1uF, Capacitor_SMD:C_0805_2012Metric, symbol Device:C
- added C22: 1uF, Capacitor_SMD:C_0805_2012Metric, symbol Device:C
- added D5: PESD1CAN, Package_TO_SOT_SMD:SOT-23-3, symbol PESD1CAN:PESD1CAN
- added FB1, FB2, FB3: FerriteBead, Resistor_SMD:R_0603_1608Metric, symbol Device:FerriteBead
- added J15: Face4, Battery Board:MOLEX_5040500591, symbol Max_Lib:Connector_Generic_Conn_01x05
- added J17: Screw_Terminal_01x02, TerminalBlock:TerminalBlock_bornier-2_P5.08mm, symbol Connector:Screw_Terminal_01x02
- added J18: I2C, Connector_JST:JST_SH_SM04B-SRSS-TB_1x04-1MP_P1.00mm_Horizontal, symbol Connector_Generic:Conn_01x04
- added J19: Screw_Terminal_01x02, Battery Board:ScrewTerminal, symbol Connector:Screw_Terminal_01x02
- added J20, J22, J26: BM04B-SRSS-TB(LF)(SN), Battery Board:JST_BM04B-SRSS-TB(LF)(SN), symbol BM04B-SRSS-TB_LF__SN_:BM04B-SRSS-TB(LF)(SN)
- added J21: CAN1, Connector_JST:JST_SH_SM04B-SRSS-TB_1x04-1MP_P1.00mm_Horizontal, symbol Connector_Generic:Conn_01x04
- added J23: CAN2, Connector_JST:JST_SH_SM04B-SRSS-TB_1x04-1MP_P1.00mm_Horizontal, symbol Connector_Generic:Conn_01x04
- added J25: Life Makes Lemonade, Connector_PinHeader_2.54mm:PinHeader_1x06_P2.54mm_Vertical, symbol Connector_Generic:Conn_01x06
- added J27: USB_B_Micro, FC_DEV_BOARD:MOLEX_105164-0001, symbol Connector:USB_B_Micro
- added JP1: SolderJumper_3_Open, Jumper:SolderJumper-3_P1.3mm_Open_RoundedPad1.0x1.5mm_NumberLabels, symbol Jumper:SolderJumper_3_Open
- added JP2: SolderJumper_2_Open, Jumper:SolderJumper-2_P1.3mm_Open_RoundedPad1.0x1.5mm, symbol Jumper:SolderJumper_2_Open
- added LED1: WS2812B_SK6812_1515, LED_SMD:LED_WS2812B_PLCC4_5.0x5.0mm_P3.2mm, symbol Adafruit ItsyBitsy RP2040-eagle-import:WS2812B_SK6805_1515
- added R31: 1-MOhm, Resistor_SMD:R_0603_1608Metric, symbol Device:R_US
- added R32, R33: 100-Ohm, Resistor_SMD:R_0603_1608Metric, symbol Device:R_US
- added R34: 10k-Ohm, Resistor_SMD:R_0603_1608Metric, symbol Device:R_US
- added R36: 1k, Resistor_SMD:R_0603_1608Metric, symbol Device:R_US
- added R39, R41: 10k, Resistor_SMD:R_0603_1608Metric, symbol mainboard:10KOHM-1_10W-1%(0603)0603
- added R45: 120, Resistor_SMD:R_0603_1608Metric, symbol mainboard:10KOHM-1_10W-1%(0603)0603
- added TP7: RESET, TestPoint:TestPoint_Loop_D1.80mm_Drill1.0mm_Beaded, symbol Connector:TestPoint
- added TP8: TestPoint, TestPoint:TestPoint_Loop_D1.80mm_Drill1.0mm_Beaded, symbol Connector:TestPoint
- added U10: MCP25625-E/ML, Package_DFN_QFN:QFN-28-1EP_6x6mm_P0.65mm_EP4.25x4.25mm, symbol MCP25625-E_ML:MCP25625-E/ML
- added U7: ADS1015IDGS, Package_SO:TSSOP-10_3x3mm_P0.5mm, symbol Analog_ADC:ADS1015IDGS
- added U8: AD8495, Package_SO:MSOP-8_3x3mm_P0.65mm, symbol Sensor_Temperature:AD8495
- added U9: TLVH431 DBZ SOT-23, Package_TO_SOT_SMD:SOT-23, symbol Reference_Voltage:TL431DBZ
- added Y2: 16MHZ 12 pf, Crystal:Crystal_SMD_2520-4Pin_2.5x2.0mm, symbol Adafruit ItsyBitsy RP2040-eagle-import:CRYSTAL2.5X2.0
- D1: renamed from D5; footprint MaxLib:PWRDI-123 -> Diode_SMD:D_PowerDI-123
- D10, D2, D3: renamed from D?; footprint Adafruit ItsyBitsy RP2040:CHIPLED_0603_NOOUTLINE -> Diode_SMD:D_0603_1608Metric_Pad1.05x0.95mm_HandSolder
- D4: renamed from D1; footprint CMSH3-40MA:DIOM5226X262N -> Diode_SMD:D_SMB
- D6: renamed from D2; footprint MaxLib:PWRDI-123 -> Diode_SMD:D_PowerDI-123
- D7: renamed from D3; footprint CMSH3-40MA:DIOM5226X262N -> Diode_SMD:D_SMB
- D8: renamed from D?; footprint Adafruit ItsyBitsy RP2040:SOD-323F -> Diode_SMD:D_SOD-323F
- D9: renamed from D4; footprint MaxLib:PWRDI-123 -> Diode_SMD:D_PowerDI-123
- IC3: renamed from IC?; footprint RO2040_Feather:QFN56_7MM_REDUCEDEPAD -> Package_DFN_QFN:QFN-56-1EP_7x7mm_P0.4mm_EP3.2x3.2mm
- IC4: renamed from IC2; footprint LT3652IMSE:SOP65P490X110-13N -> Package_SO:MSOP-12-1EP_3x4mm_P0.65mm_EP1.65x2.85mm
- J10: renamed from J1; footprint MOLEX PICO LOCK 5 POS:MOLEX_5040500591 -> Battery Board:MOLEX_5040500591
- J11: renamed from J2; footprint MOLEX PICO LOCK 5 POS:MOLEX_5040500591 -> Battery Board:MOLEX_5040500591
- J12: renamed from J3; footprint MOLEX PICO LOCK 5 POS:MOLEX_5040500591 -> Battery Board:MOLEX_5040500591
- J13: renamed from J4; footprint MOLEX PICO LOCK 5 POS:MOLEX_5040500591 -> Battery Board:MOLEX_5040500591
- J14: renamed from J5; footprint MOLEX PICO LOCK 5 POS:MOLEX_5040500591 -> Battery Board:MOLEX_5040500591
- J16: renamed from J7; footprint (none) -> Connector_JST:JST_SH_SM04B-SRSS-TB_1x04-1MP_P1.00mm_Horizontal
- J2: renamed from J19; footprint MOLEX PICO LOCK 2 POS:MOLEX_504050-0291 -> Battery Board:MOLEX_504050-0291
- J24: renamed from J?; footprint RO2040_Feather:2X05_1.27MM_BOX_POSTS -> Battery Board:JTAG_2X05_1.27MM_BOX_NOCREAM
- J3: renamed from J17; footprint MOLEX PICO LOCK 2 POS:MOLEX_504050-0291 -> Battery Board:MOLEX_504050-0291
- J4: renamed from J11; footprint MOLEX PICO LOCK 2 POS:MOLEX_504050-0291 -> Battery Board:MOLEX_504050-0291
- J5: renamed from J12; footprint MOLEX PICO LOCK 2 POS:MOLEX_504050-0291 -> Battery Board:MOLEX_504050-0291
- J6: renamed from J13; footprint MOLEX PICO LOCK 2 POS:MOLEX_504050-0291 -> Battery Board:MOLEX_504050-0291
- J7: renamed from J14; footprint MOLEX PICO LOCK 2 POS:MOLEX_504050-0291 -> Battery Board:MOLEX_504050-0291
- J8: renamed from J15; footprint MOLEX PICO LOCK 2 POS:MOLEX_504050-0291 -> Battery Board:MOLEX_504050-0291
- J9: renamed from J16; footprint MOLEX PICO LOCK 2 POS:MOLEX_504050-0291 -> Battery Board:MOLEX_504050-0291
- Q6: renamed from Q5; footprint MaxLib:SOT-23 -> Package_TO_SOT_SMD:SOT-23
- Q7: renamed from Q8; footprint MaxLib:SOT-23 -> Package_TO_SOT_SMD:SOT-23
- Q8: renamed from Q6; footprint MaxLib:NDS8434 -> Package_SO:SOIC-8-1EP_3.9x4.9mm_P1.27mm_EP2.514x3.2mm
- Q9: footprint MaxLib:NDS8434 -> Package_SO:SOIC-8-1EP_3.9x4.9mm_P1.27mm_EP2.514x3.2mm
- SW1, SW2: renamed from SW?; footprint Adafruit ItsyBitsy RP2040:BTN_KMR2_4.6X2.8 -> Battery Board:BTN_KMR2_4.6X2.8
- U1: footprint R5460N233AF:R5460N233AF-SOT95P280X130-6N -> Package_TO_SOT_SMD:SOT-23-6
- U3: renamed from U2; footprint MaxLib:PWP14_2P31X2P46-L -> Package_SO:HTSSOP-14-1EP_4.4x5mm_P0.65mm_EP3.4x5mm_Mask3x3.1mm_ThermalVias
- U6: renamed from U5; footprint MaxLib:TPS7A4501DCQT -> Package_TO_SOT_SMD:SOT-223-6
- Y1: renamed from Y?; footprint Adafruit ItsyBitsy RP2040:CRYSTAL_2.5X2 -> Crystal:Crystal_SMD_2520-4Pin_2.5x2.0mm
- gave numbers to parts that had none: 24
- renumbered C15 to C13, C13 to C14, C19 to C15, C16 to C34, C17 to C39, C18 to C40, C20 to C41, C14 to C42, IC3 to IC2, J18 to J1, Q7 to Q4, Q4 to Q5, R8 to R10, R9 to R11, R10 to R12, R11 to R13, R12 to R14, R13 to R15, R15 to R17, R44 to R19, R38 to R2, R24 to R20, R14 to R21, R40 to R22, R16 to R23, R41 to R24, R30 to R25, R31 to R26, R17 to R27, R42 to R28, R28 to R29, R2 to R3, R29 to R30, R3 to R4, R32 to R42, R33 to R43, R43 to R46, R37 to R48, R22 to R49, R4 to R5, R34 to R50, R35 to R51, R36 to R54, R5 to R6, R6 to R7, R7 to R8, R39 to R9, TP5 to TP1, TP1 to TP2, TP2 to TP3, TP3 to TP4, TP4 to TP5, U6 to U11, U3 to U13, U7 to U2, U8 to U4, U4 to U5
Connections:
- net RF1_IO0 is gone; now on net CHRG': IC3.35 (GPIO23)
- net SCL_FC is gone; now on net SCL0: U5.22 (SCL)
- net SDA_FC is gone; now on net SDA0: U5.23 (SDA)
- net +3V3: now also C24.2, FB1.2, FB2.2, J15.3 (Pin_3), J18.2 (Pin_2), J20.1, J21.2 (Pin_2), J23.2 (Pin_2), J25.6 (Pin_6), JP1.1 (A), JP2.2 (B), R39.1, R41.1, U10.11 (VIO), U10.3 (VDD@1)
- net FC_RESET: now also IC1.12 (LED6), J15.4 (Pin_4)
- net FC_RX: now also J25.2 (Pin_2)
- net FC_TX: now also J25.3 (Pin_3)
- net GND: now also IC3.57 (GND), C13.1, C13.2, C13.2, C13.2, C17.1, C19.2, C22.2, C24.1, D5.3, FB3.2, J15.2 (Pin_2), J15.5 (Pin_5), J18.1 (Pin_1), J20.2, J20.4, J20.S1 (SHIELD), J20.S2 (SHIELD), J21.1 (Pin_1), J22.S1 (SHIELD), J22.S2 (SHIELD), J23.1 (Pin_1), J25.1 (Pin_1), J26.4, J26.S1 (SHIELD), J26.S2 (SHIELD), J27.5 (GND), J27.SH1 (Shield), LED1.3 (GND), R31.2, R34.1, U10.15 (STBY), U10.18 (VSS@1), U10.22 (GND), U10.29 (GND@1), U8.3 (-Vs), U9.3 (A); no longer IC3.P$1 (GND)
- net NEOPIX: now also LED1.4 (DI)
- net NEO_PWR: now also LED1.1 (VDD)
- net SCL0: now also U7.10 (SCL)
- net SCL1: now also J18.4 (Pin_4), J25.4 (Pin_4)
- net SDA0: now also U7.9 (SDA)
- net SDA1: now also J18.3 (Pin_3), J25.5 (Pin_5)
- net SPI0_CS0: now also IC3.12 (GPIO9), R41.2, U10.1 (CS); no longer IC3.28 (GPIO17)
- net SPI0_MISO: now also IC3.11 (GPIO8), U10.28 (SO); no longer IC3.27 (GPIO16)
- net SPI0_MOSI: now also IC3.14 (GPIO11), U10.27 (SI); no longer IC3.30 (GPIO19)
- net SPI0_SCK: now also IC3.13 (GPIO10), U10.26 (SCK); no longer IC3.29 (GPIO18)
- net SPI1_CS0: now also IC3.28 (GPIO17), J22.1; no longer IC3.12 (GPIO9)
- net SPI1_MISO: now also IC3.27 (GPIO16), J22.4; no longer IC3.11 (GPIO8)
- net SPI1_MOSI: now also IC3.30 (GPIO19), J22.3; no longer IC3.14 (GPIO11)
- net SPI1_SCK: now also IC3.29 (GPIO18), J22.2; no longer IC3.13 (GPIO10)
- net USBBOOT: now also TP8.1
- net VBUS: now also J26.1, J27.1 (VBUS)
- net V_RF: now also JP1.3 (B)
- net at R52.2: now also J27.3 (D+)
- net at R53.2: now also J27.2 (D-)
- net D+ renamed USB_D+
- net USB_D+: now also J26.3
- net D- renamed USB_D-
- net USB_D-: now also J26.2
- net EEPROM_CONTROL renamed D0
- net EEPROM_POWER renamed D1
- net XSHUT renamed A0
- new net: JP2.1 (A), R34.2, U7.1 (ADDR)
- new net: R36.1, U8.2 (REF), U9.1 (K), U9.2 (REF)
- new net: C22.1, FB1.1, R36.2, U8.7 (+Vs)
- new net: C13.1, U10.21 (OSC1), Y2.3 (2)
- new net: R39.2, TP7.1, U10.2 (RESET)
- new net: C13.1, U10.20 (OSC2), Y2.1
- new net: J17.1 (Pin_1), J19.2 (Pin_2), R31.1, R33.2
- new net: J17.2 (Pin_2), J19.1 (Pin_1), R32.1
- new net: C18.1, C19.1, R33.1, U8.8 (+IN)
- new net: C17.2, C18.2, R32.2, U8.1 (-IN)
- new net +5V: J15.1 (Pin_1), J20.3, JP1.2 (C), U10.19 (VDDA)
- new net AGND: C16.2, C27.2, FB3.1, U7.3 (GND)
- new net AVDD: C16.1, C27.1, FB2.1, U7.4 (AIN0), U7.6 (AIN2), U7.7 (AIN3), U7.8 (VDD)
- new net CANH: C13.2, D5.2, J21.4 (Pin_4), J23.4 (Pin_4), R45.2, U10.13 (CANH)
- new net CANL: C13.1, D5.1, J21.3 (Pin_3), J23.3 (Pin_3), R45.1, U10.12 (CANL)
- new net OUT: U7.5 (AIN1), U8.5 (SENSE), U8.6
- new net RXCAN: U10.10 (RXD), U10.5 (RXCAN)
- new net TXCAN: U10.16 (TXD), U10.4 (TXCAN)
- no-connect marks 30 -> 39
Other:
- note added: "Default I2C: 0x48"
- note added: "Jumped I2C: 0x49"
- moved on the sheet: D10, R56
