File: battery_board_v3b/battery_board_v3b.kicad_pcb (KiCad board)
At the start: 4 copper layers, 88 x 94.5 mm, 204 parts, among them IC2 PCT2075DP,118, IC3 RP2040_QFN56, IC4 LT3652IMSE#PBF, J1 Bypass, J10 Jetson, J11 BM04B-SRSS-TB(LF)(SN), J14 Solar, J15 FC, J16 I2C Multiplexer Breakout, J17 ISS Foot, J18 Screw_Terminal_01x02, J19 BM04B-SRSS-TB(LF)(SN), J2 Heater, J20 CAN1, J21 BM04B-SRSS-TB(LF)(SN), J22 CAN2, J23 Conn_ARM_JTAG_SWD_10, J24 USB_B_Micro, J25 Life Makes Lemonade, J26 BM04B-SRSS-TB(LF)(SN), J27 I2C0 Breakout, J3 BURN, J4 CHARGE, J5 Foot0, J6 Foot1, J7 Foot2, J8 Foot3, J9 RBF, K1 APAN3105, Q1 IRF7458, Q10 IRLML2803, Q11 NDS8434, Q2 IRF7458, Q3 MBT2222ADW1T1, Q4 MMBT2222AT, Q5 MBT2222ADW1T1, Q6 IRLML2803, Q7 IRLML2803, Q8 NDS8434, Q9 NDS8434, SW1 KMR2, SW2 KMR2, U1 R5460N208AA, U10 TLVH431 DBZ SOT-23, U11 MCP25625-E/ML, U12 INA219AxD, U13 MAX706RESA, U14 INA219AxD, U2 1049, U3 TPS54226PWPRPWP14_2P31X2P46-L, U4 1049, U5 TPS54226PWPRPWP14_2P31X2P46-L, U6 TPS7A4501DCQT, U7 ADS1015IDGS, U8 W25Q128JV, U9 AD8495, Y1 Crystal_GND24, Y2 Crystal_GND24

Commit message: Updated JST Connectors to be All One Footprint
Parts:
- J16, J20, J22: footprint Connector_JST:JST_SH_SM04B-SRSS-TB_1x04-1MP_P1.00mm_Horizontal -> Battery Board:JST_BM04B-SRSS-TB(LF)(SN)
- moved J16 1.26 mm to (117.2, 106.4)
- moved J20 0.73 mm to (172.2, 46.0)
- moved J22 0.73 mm to (180.2, 46.0)
Routing:
- net +3V3: track 60.7 -> 72.5 mm, vias 25 -> 26
- net GND: track 314.7 -> 322.5 mm
- net CANH: track 30.7 -> 38.3 mm
- net CANL: track 30.9 -> 38.5 mm
- net SDA0: track 162.5 -> 165.7 mm
- net SCL0: track 159.1 -> 162.4 mm
