File: inhibit_diagram/inhibit_diagram.kicad_sch (KiCad schematic)
At the start: 10 parts

Commit message: Updated Inhibit Diagram to Reflect V3
Parts:
- added Foot6: SW_Push_Open, symbol Switch:SW_Push_Open
- renumbered ISSFoot1 to Foot5
Connections:
- net at BT1.2 (-), Foot5.1 (A), SC1.2 (-): now also Foot6.1 (A)
- net at Foot5.2 (B), R1.2: now also Foot6.2 (B)
Other:
- note added: "March 31, 2025 Drafted by: Michael Pham"
- note added: "PROVES V3 Battery Inhibit Scheme Simplified View Battery Protection and Power Regulation Not Shown"
- note removed: "PROVES V1.5 Battery Inhibit Scheme Simplified View Battery Protection and Power Regulation Not Shown"
- note removed: "September 25, 2024 Drafted by: Michael Pham"
- moved on the sheet: Foot5
Changed lines of the file:
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@@
 (kicad_sch
-	(version 20231120)
+	(version 20250114)
 	(generator "eeschema")
-	(generator_version "8.0")
+	(generator_version "9.0")
 	(paper "A5")
+	(text "Remove Before \nFlight Pin"
+		(exclude_from_sim no)
+		(at 146.558 34.544 0)
+		(effects
+			(font
+				(size 1.27 1.27)
+			)
+		)
+	)
+	(text "PROVES V3 Battery Inhibit Scheme Simplified View\nBattery Protection and Power Regulation Not Shown"
+		(exclude_from_sim no)
+		(at 65.786 21.59 0)
+		(effects
+			(font
+				(size 1.27 1.27)
+			)
+		)
+	)
+	(text "All inhibits are wired as normally closed\nand thrown open when in deployer."
+		(exclude_from_sim no)
+		(at 106.934 63.754 0)
+		(effects
+			(font
+				(size 1.27 1.27)
+			)
+		)
+	)
+	(text "March 31, 2025\nDrafted by: Michael Pham"
+		(exclude_from_sim no)
+		(at 151.384 86.614 0)
+		(effects
+			(font
+				(size 1.27 1.27)
+			)
+		)
+	)
+	(text "High Side Foot Switch Inhibit"
+		(exclude_from_sim no)
+		(at 106.934 28.448 0)
+		(effects
+			(font
+				(size 1.27 1.27)
+			)
+		)
+	)
+	(text "Low Side Foot Switch Inhibit"
+		(exclude_from_sim no)
+		(at 106.172 84.836 0)
+		(effects
+			(font
+				(size 1.27 1.27)
+			)
+		)
+	)
+	(junction
+		(at 111.76 78.74)
+		(diameter 0)
+		(color 0 0 0 0)
+	)
 	(junction
 		(at 83.82 45.72)
@@
 	)
 	(junction
+		(at 101.6 78.74)
+		(diameter 0)
+		(color 0 0 0 0)
+	)
+	(junction
 		(at 130.81 45.72)
 		(diameter 0)
@@
 	(wire
 		(pts
+			(xy 111.76 78.74) (xy 111.76 81.28)
+		)
+		(stroke
+			(width 0)
+			(type default)
+		)
+	)
+	(wire
+		(pts
 			(xy 160.02 66.04) (xy 160.02 78.74)
 		)
@@
 		)
 	)
+	(wire
+		(pts
+			(xy 101.6 78.74) (xy 101.6 81.28)
+		)
+		(stroke
+			(width 0)
+			(type default)
+		)
+	)
 	(polyline
 		(pts
@@
 		)
 	)
+	(wire
+		(pts
+			(xy 101.6 76.2) (xy 101.6 78.74)
+		)
+		(stroke
+			(width 0)
+			(type default)
+		)
+	)
 	(polyline
 		(pts
@@
 		)
 	)
-	(text "Remove Before \nFlight Pin"
-		(exclude_from_sim no)
-		(at 146.558 34.544 0)
-		(effects
-			(font
-				(size 1.27 1.27)
-			)
-		)
-	)
-	(text "PROVES V1.5 Battery Inhibit Scheme Simplified View\nBattery Protection and Power Regulation Not Shown"
-		(exclude_from_sim no)
-		(at 65.786 21.59 0)
-		(effects
-			(font
-				(size 1.27 1.27)
-			)
-		)
-	)
-	(text "All inhibits are wired as normally closed\nand thrown open when in deployer."
-		(exclude_from_sim no)
-		(at 106.934 63.754 0)
-		(effects
-			(font
-				(size 1.27 1.27)
-			)
-		)
-	)
-	(text "September 25, 2024\nDrafted by: Michael Pham"
-		(exclude_from_sim no)
-		(at 151.384 86.614 0)
-		(effects
-			(font
-				(size 1.27 1.27)
-			)
-		)
-	)
-	(text "High Side Foot Switch Inhibit"
-		(exclude_from_sim no)
-		(at 106.934 28.448 0)
-		(effects
-			(font
-				(size 1.27 1.27)
-			)
-		)
-	)
-	(text "Low Side Foot Switch Inhibit"
-		(exclude_from_sim no)
-		(at 106.172 84.836 0)
-		(effects
-			(font
-				(size 1.27 1.27)
-			)
+	(wire
+		(pts
+			(xy 111.76 76.2) (xy 111.76 78.74)
+		)
+		(stroke
+			(width 0)
+			(type default)
 		)
 	)
@@
 	(symbol
 		(lib_id "Switch:SW_Push_Open")
+		(at 106.68 81.28 0)
+		(unit 1)
+		(exclude_from_sim no)
+		(in_bom yes)
+		(on_board yes)
+		(dnp no)
+		(property "Reference" "Foot6"
+			(at 96.266 81.28 0)
+			(effects
+				(font
+					(size 1.27 1.27)
+				)
+			)
+		)
+		(property "Value" "SW_Push_Open"
+			(at 121.412 81.28 0)
+			(effects
+				(font
+					(size 1.27 1.27)
+				)
+			)
+		)
+		(property "Footprint" ""
+			(at 106.68 76.2 0)
+			(effects
+				(font
+					(size 1.27 1.27)
+				)
+				(hide yes)
+			)
+		)
+		(property "Datasheet" "~"
+			(at 106.68 76.2 0)
+			(effects
+				(font
+					(size 1.27 1.27)
+				)
+				(hide yes)
+			)
+		)
+		(property "Description" "Push button switch, push-to-open, generic, two pins"
+			(at 106.68 81.28 0)
+			(effects
+				(font
+					(size 1.27 1.27)
+				)
+				(hide yes)
+			)
+		)
+		(pin "1"
+		)
+		(pin "2"
+		)
+		(instances
+			(project "inhibit_diagram"
+				(path "/0befa4ae-1f61-40ba-9027-ba4deb5af2e8"
+					(reference "Foot6")
+					(unit 1)
+				)
+			)
+		)
+	)
+	(symbol
+		(lib_id "Switch:SW_Push_Open")
 		(at 146.05 45.72 0)
 		(unit 1)
@@
 	(symbol
 		(lib_id "Switch:SW_Push_Open")
-		(at 106.68 78.74 0)
+		(at 106.68 76.2 0)
 		(unit 1)
 		(exclude_from_sim no)
@@
 		(on_board yes)
 		(dnp no)
-		(fields_autoplaced yes)
-		(property "Reference" "ISSFoot1"
-			(at 106.68 72.39 0)
+		(property "Reference" "Foot5"
+			(at 96.266 76.2 0)
 			(effects
 				(font
@@
 		)
 		(property "Value" "SW_Push_Open"
-			(at 106.68 74.93 0)
+			(at 121.412 75.946 0)
 			(effects
 				(font
@@
 		)
 		(property "Footprint" ""
-			(at 106.68 73.66 0)
+			(at 106.68 71.12 0)
 			(effects
 				(font
@@
 		)
 		(property "Datasheet" "~"
-			(at 106.68 73.66 0)
+			(at 106.68 71.12 0)
 			(effects
 				(font
@@
 		)
 		(property "Description" "Push button switch, push-to-open, generic, two pins"
-			(at 106.68 78.74 0)
+			(at 106.68 76.2 0)
 			(effects
 				(font
@@
 			(project "inhibit_diagram"
 				(path "/0befa4ae-1f61-40ba-9027-ba4deb5af2e8"
-					(reference "ISSFoot1")
+					(reference "Foot5")
 					(unit 1)
 				)
@@
 		)
 	)
+	(embedded_fonts no)
 )
